Commit message: add inertial to m900ia

File: fanuc_m900ia_support/urdf/m900ia260l_macro.xacro (robot description, xacro)
@@ -2,4 +2,7 @@
 <robot xmlns:xacro="http://wiki.ros.org/xacro">
   <xacro:include filename="$(find fanuc_resources)/urdf/common_materials.xacro"/>
+  <xacro:property name="density" value="1048" />
+  <xacro:property name="scaling" value="0.00001" />
+  <xacro:property name="dens_scale" value="${density}*${scaling}" />
   <xacro:macro name="fanuc_m900ia260l" params="prefix">
     <!-- links: main serial chain -->
@@ -18,4 +21,12 @@
         </geometry>
       </collision>
+      <inertial>
+        <origin xyz="-0.0479547 0.0005924 0.1838477 " rpy="0 0 0"/>
+        <mass value="0.179502640*{density}"/>
+        <inertia
+          ixx="758.002563*${dens_scale}" ixy="0.059074*${dens_scale}" ixz="-29.833698*${dens_scale}"
+          iyy="1059.352539*${dens_scale}" iyz="0.779661*${dens_scale}"
+          izz="1392.725098*${dens_scale}"/>
+      </inertial>
     </link>
     <link name="${prefix}link_1">
@@ -33,4 +44,12 @@
         </geometry>
       </collision>
+      <inertial>
+        <origin xyz="0.2508056 -0.0039480 -0.1876394 " rpy="0 0 0"/>
+        <mass value="0.428307129*{density}"/>
+        <inertia
+          ixx="4593.856934*${dens_scale}" ixy="-51.459423*${dens_scale}" ixz="-767.660156*${dens_scale}"
+          iyy="3659.617188*${dens_scale}" iyz="0.543368*${dens_scale}"
+          izz="4472.774902*${dens_scale}"/>
+      </inertial>
     </link>
     <link name="${prefix}link_2">
@@ -48,4 +67,12 @@
         </geometry>
       </collision>
+      <inertial>
+        <origin xyz="0.0208002 -0.0321524 0.4698709 " rpy="0 0 0"/>
+        <mass value="0.146323502*{density}"/>
+        <inertia
+          ixx="1881.386841*${dens_scale}" ixy="-15.604090*${dens_scale}" ixz="29.171331*${dens_scale}"
+          iyy="1862.439209*${dens_scale}" iyz="-94.617111*${dens_scale}"
+          izz="311.525116*${dens_scale}"/>
+      </inertial>
     </link>
     <link name="${prefix}link_3">
@@ -63,4 +90,12 @@
         </geometry>
       </collision>
+      <inertial>
+        <origin xyz="0.3940928 -0.0020985 0.1485200" rpy="0 0 0"/>
+        <mass value="0.206138123*{density}"/>
+        <inertia
+          ixx="399.825439*${dens_scale}" ixy="2.884355*${dens_scale}" ixz="-246.776382*${dens_scale}"
+          iyy="5650.399902*${dens_scale}" iyz="-2.081667*${dens_scale}"
+          izz="5621.276855*${dens_scale}"/>
+      </inertial>
     </link>
     <link name="${prefix}link_4">
@@ -78,4 +113,12 @@
         </geometry>
       </collision>
+      <inertial>
+        <origin xyz="1.5984120 -0.0070510 -0.0000020" rpy="0 0 0"/>
+        <mass value="0.011438374*{density}"/>
+        <inertia
+          ixx="6.721434*${dens_scale}" ixy="0.585065*${dens_scale}" ixz="-0.000148*${dens_scale}"
+          iyy="14.125363*${dens_scale}" iyz="-0.000006*${dens_scale}"
+          izz="13.054061*${dens_scale}"/>
+      </inertial>
     </link>
     <link name="${prefix}link_5">
@@ -93,4 +136,12 @@
         </geometry>
       </collision>
+      <inertial>
+        <origin xyz="0.0419062 -0.0278710 -0.0000007" rpy="0 0 0"/>
+        <mass value="0.020431719*{density}"/>
+        <inertia
+          ixx="22.334682*${dens_scale}" ixy="-2.872280*${dens_scale}" ixz="0.000051*${dens_scale}"
+          iyy="24.979155*${dens_scale}" iyz="0.000064*${dens_scale}"
+          izz="29.386639*${dens_scale}"/>
+      </inertial>
     </link>
     <link name="${prefix}link_6">
@@ -108,4 +159,12 @@
         </geometry>
       </collision>
+      <inertial>
+        <origin xyz="-0.0274942 -0 -0" rpy="0 0 0"/>
+        <mass value="0.002406848*{density}"/>
+        <inertia
+          ixx="1.555723*${dens_scale}" ixy="0*${dens_scale}" ixz="0*${dens_scale}"
+          iyy="0.850091*${dens_scale}" iyz="0.0000*${dens_scale}"
+          izz="0.850086*${dens_scale}"/>
+      </inertial>
     </link>
     <!-- joints: main serial chain -->
@@ -167,4 +226,12 @@
         </geometry>
       </collision>
+      <inertial>
+        <origin xyz="-0.1043124 -0.0504379 -0.0145418" rpy="0 0 0"/>
+        <mass value="0.027578537*{density}"/>
+        <inertia
+          ixx="32.950230*${dens_scale}" ixy="-1.911048*${dens_scale}" ixz="-1.272046*${dens_scale}"
+          iyy="97.812645*${dens_scale}" iyz="0.253856*${dens_scale}"
+          izz="73.873703*${dens_scale}"/>
+      </inertial>
     </link>
     <link name="${prefix}plink_2">
@@ -182,4 +249,12 @@
         </geometry>
       </collision>
+      <inertial>
+        <origin xyz="-0.0285391 0.0022351 -0.5422898" rpy="0 0 0"/>
+        <mass value="0.012706021*{density}"/>
+        <inertia
+          ixx="115.503403*${dens_scale}" ixy="-0.027600*${dens_scale}" ixz="-1.782988*${dens_scale}"
+          iyy="118.431725*${dens_scale}" iyz="-0.022260*${dens_scale}"
+          izz="3.922133*${dens_scale}"/>
+      </inertial>
     </link>
     <joint name="${prefix}pjoint_1" type="continuous">
